Commit message: simulation_pkg

File: src/simulation_pkg/urdf/turtlebot3_burger.urdf (robot description, URDF)
Before this commit: robot turtlebot3_burger, 7 links, 6 joints
Links:
- link ${namespace}base_link: geometry collision box size=0.140 0.140 0.143; visual geometry 

Commit message: testing

File: src/simulation_pkg/urdf/turtlebot3_burger.urdf (robot description, URDF)
Before this commit: robot turtlebot3_burger, 7 links, 6 joints
Links:
- link ${namespace}base_link: geometry collision box size=0.140 0.140 0.143; visual mesh filename=package://turtlebot3_description/meshes/bases/burger_base.s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 scale=0.001 0.001 0.001
